File: Borealis/Borealis/Borealis.kicad_sch (KiCad schematic)
At the start: 0 parts

Commit message: Remove Mainboard_prototype and update schematic
Parts:
- added J1: Conn_01x06_Pin, symbol Connector:Conn_01x06_Pin
- added J3: Conn_01x02_Pin, symbol Connector:Conn_01x02_Pin
- added J4: Conn_01x08_Pin, symbol Connector:Conn_01x08_Pin
- added R1, R2, R3: R, symbol Device:R
- added U1: Pico, RPi_Pico:RPi_Pico_SMD_TH, symbol MCU_RaspberryPi_and_Boards:Pico
Connections:
- new net: J4.1 (Pin_1), U1.3 (GND)
- new net: J1.2 (Pin_2), J4.2 (Pin_2), U1.37 (3V3_EN)
- new net: J1.4 (Pin_4), J4.3 (Pin_3), U1.2 (GPIO1)
- new net: J1.5 (Pin_5), J4.4 (Pin_4), U1.1 (GPIO0)
- new net: J4.5 (Pin_5), R1.1
- new net: J4.6 (Pin_6), R2.1
- new net: J4.7 (Pin_7), U1.20 (GPIO15)
- new net: J3.1 (Pin_1), J4.8 (Pin_8)
- new net: J1.1 (Pin_1), R3.2, U1.38 (GND)
- new net: J1.3 (Pin_3), J3.2 (Pin_2), U1.40 (VBUS)
- new net: J1.6 (Pin_6), R3.1, U1.32 (GPIO27_ADC1)
- new net: R1.2, U1.21 (GPIO16)
- new net: R2.2, U1.22 (GPIO17)
