File: Borealis/sensor-board-solar/sensor-board-solar.kicad_sch (KiCad schematic)
At the start: 0 parts

Commit message: added solar sensor module
Parts:
- added A1: ADS1115_ADC_Module, Charleslabs_Parts:ADC1115_ADC_Module, symbol Charleslabs_Parts:ADS1115_ADC_Module
- added J1: Conn_01x06_Pin, symbol Connector:Conn_01x06_Pin
- added J2: Conn_01x02_Pin (solar), Connector_JST:JST_JWPF_B02B-JWPF-SK-R_1x02_P2.00mm_Vertical, symbol Connector:Conn_01x02_Pin
- added R1: R, symbol Device:R
Connections:
- new net: J1.6 (Pin_6), R1.2
- new net +3.3V: A1.1 (VCC), J1.2 (Pin_2), R1.1
- new net GND: A1.2 (GND), J1.1 (Pin_1), J2.2 (Pin_2)
- new net SCL: A1.3 (SCL), J1.4 (Pin_4)
- new net SDA: A1.4 (SDA), J1.5 (Pin_5)
- new net analog: A1.7 (A0), J2.1 (Pin_1)
