File: Borealis/sensor-board-solar/sensor-board-solar.kicad_sch (KiCad schematic)
At the start: 7 parts, among them J1 Conn_01x02_Pin (Solar panel c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, J2 Conn_01x03_Pin (data connecti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, J5 Conn_01x03_Pin (power connect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

Commit message: Fixed a few things
Parts:
- removed ADS1115IDGSR1: ~, batteryholder:ADS1115IDGSR, symbol ADS1115IDGSR_2025-12-25-altium-import:root_0_ADS1115IDGSR_
- removed J2: Conn_01x03_Pin (data connection to main board), batteryholder:1x03 2.3 pitch, symbol Connector:Conn_01x03_Pin
- removed J5: Conn_01x03_Pin (power connection to main board), batteryholder:1x03 2.3 pitch, symbol Connector:Conn_01x03_Pin
- added J4, J7: 878-22-004-10-011101, BOREALIS:8782200410011101, symbol 878-22-004-10-011101:878-22-004-10-011101
Connections:
- net Solar_Analog is gone; now on net ADC: R2.1, R3.2
- net +3.3V: now also J4.2
- net +5V: now also J4.3
- net ADC: now also J7.3; no longer R1.2
- net GND: now also J4.1
- net SCL: now also J7.1
- net SDA: now also J7.2
- new net ID: J4.4, R1.2
- no-connect marks 5 -> 1
Other:
- moved on the sheet: J1, R2, R3

Commit message: Worked on sum stuff
Parts:
- removed J4, J7: 878-22-004-10-011101, BOREALIS:8782200410011101, symbol 878-22-004-10-011101:878-22-004-10-011101
- added U1, U2: MAGNETIC POGO CONN., batteryholder:MAGNETIC POGO CONN., symbol magnetic_pogo_conn.:MAGNETIC_POGO_CONN.
- J1: footprint Connector_PinHeader_2.54mm:PinHeader_1x02_P2.54mm_Vertical -> Connector_JST:JST_PH_B2B-PH-K_1x02_P2.00mm_Vertical
Connections:
- net +3.3V: now also U2.2
- net +5V: now also U2.3
- net ADC: now also U1.2
- net GND: now also U2.1
- net ID: now also U2.4
- net SCL: now also U1.4
- net SDA: now also U1.3
Other:
- moved on the sheet: J1, R2, R3

Commit message: Worked on boards
Parts:
- added H1: MountingHole, MountingHole:MountingHole_2.7mm_M2.5_Pad, symbol Mechanical:MountingHole
Changed lines of the file:
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@@
+	)
+	(symbol
+		(lib_id "Mechanical:MountingHole")
+		(at 85.09 142.24 0)
+		(unit 1)
+		(exclude_from_sim no)
+		(in_bom no)
+		(on_board yes)
+		(dnp no)
+		(fields_autoplaced yes)
+		(property "Reference" "H1"
+			(at 87.63 140.9699 0)
+			(effects
+				(font
+					(size 1.27 1.27)
+				)
+				(justify left)
+			)
+		)
+		(property "Value" "MountingHole"
+			(at 87.63 143.5099 0)
+			(effects
+				(font
+					(size 1.27 1.27)
+				)
+				(justify left)
+			)
+		)
+		(property "Footprint" "MountingHole:MountingHole_2.7mm_M2.5_Pad"
+			(at 85.09 142.24 0)
+			(effects
+				(font
+					(size 1.27 1.27)
+				)
+				(hide yes)
+			)
+		)
+		(property "Datasheet" "~"
+			(at 85.09 142.24 0)
+			(effects
+				(font
+					(size 1.27 1.27)
+				)
+				(hide yes)
+			)
+		)
+		(property "Description" "Mounting Hole without connection"
+			(at 85.09 142.24 0)
+			(effects
+				(font
+					(size 1.27 1.27)
+				)
+				(hide yes)
+			)
+		)
+		(instances
+			(project ""
+				(path "/31536c3d-d3f9-4dfb-892e-75fc519025d6"
+					(reference "H1")
+					(unit 1)
+				)
+			)
+		)
 	)
 	(symbol
