File: Borealis/sensor-board-solar/sensor-board-solar.kicad_pcb (KiCad board)
At the start: 2 copper layers, 20 x 20 mm, 7 parts, among them J1 Conn_01x02_Pin (Solar panel c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, J2 Conn_01x03_Pin (data connecti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, J5 Conn_01x03_Pin (power connect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

Commit message: Worked on sum stuff
Parts:
- removed ADS1115IDGSR1: ~, batteryholder:ADS1115IDGSR
- removed J2: Conn_01x03_Pin (data connection to main board), batteryholder:1x03 2.3 pitch
- removed J5: Conn_01x03_Pin (power connection to main board), batteryholder:1x03 2.3 pitch
- added U1: MAGNETIC POGO CONN., batteryholder:MAGNETIC POGO CONN., F.Cu at (149.0, 83.8)
- added U2: MAGNETIC POGO CONN., batteryholder:MAGNETIC POGO CONN., F.Cu at (132.0, 83.8)
- J1: footprint Connector_PinHeader_2.54mm:PinHeader_1x02_P2.54mm_Vertical -> Connector_JST:JST_PH_B2B-PH-K_1x02_P2.00mm_Vertical; moved to B.Cu
- moved J1 63.6 mm to (141.4, 85.0), turned to 180 degrees
- moved R2 61.7 mm to (143.4, 79.0), turned to -90 degrees
- moved R3 61.6 mm to (140.4, 79.0), turned to 90 degrees
- moved R1 48.4 mm to (137.4, 79.0)
Connections:
- R1 pad 2: /ADC -> /ID
- R2 pad 1: /Solar_Analog -> /ADC
- R3 pad 2: /Solar_Analog -> /ADC
Routing:
- net +3.3V: track 30.5 -> 7.84 mm
- net /SCL: track 10.4 -> 0.00 mm
- net /SDA: track 9.03 -> 0.00 mm
- net /ADC: track 2.50 -> 10.2 mm
- net GND: track 20.9 -> 14.6 mm
- net /Solar_Analog: track 6.03 -> 0.00 mm
- net /ID: track 0.00 -> 5.62 mm
- net Net-(J1-Pin_1): track 7.88 -> 5.92 mm
Other:
- board size 20 x 20 mm -> 23.6 x 23.5 mm
- board text removed: "Borealis Sensor Board Solar panel"

Commit message: Worked on boards
Parts:
- added H1: MountingHole, MountingHole:MountingHole_2.7mm_M2.5_Pad, F.Cu at (140.4, 92.6)
Other:
- outline, holes or cut-outs redrawn
- board text added: "Borealis Voltmeter"
