File: Borealis/sensor-board-ozone/sensor-board-ozone.kicad_sch (KiCad schematic)
At the start: 7 parts, among them J1 Conn_01x02_Pin (Solar panel c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, J2 Conn_01x03_Pin (data connecti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, J5 Conn_01x03_Pin (power connect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

Commit message: Fixed a few things
Parts:
- removed ADS1115IDGSR1: ~, batteryholder:ADS1115IDGSR, symbol ADS1115IDGSR_2025-12-25-altium-import:root_0_ADS1115IDGSR_
- removed J1: Conn_01x02_Pin (Solar panel connection), symbol Connector:Conn_01x02_Pin
- removed J2: Conn_01x03_Pin (data connection to main board), symbol Connector:Conn_01x03_Pin
- removed J5: Conn_01x03_Pin (power connection to main board), symbol Connector:Conn_01x03_Pin
- added J2: Conn_01x04_Pin (MQ series sensor. 4pins (5v, gnd,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, symbol Connector:Conn_01x04_Pin
- added J4, J7: 878-22-004-10-011101, BOREALIS:8782200410011101, symbol 878-22-004-10-011101:878-22-004-10-011101
- R1: footprint OptoDevice:R_LDR_4.9x4.2mm_P2.54mm_Vertical -> Resistor_SMD:R_0805_2012Metric
- R2, R3: footprint (none) -> Resistor_SMD:R_0805_2012Metric
Connections:
- net Solar_Analog is gone; now on net ADC: R2.1, R3.2
- net +3.3V: now also J4.2
- net +5V: now also J2.1 (Pin_1), J4.3
- net ADC: now also J7.3; no longer R1.2
- net GND: now also J2.2 (Pin_2), J4.1
- net SCL: now also J7.1
- net SDA: now also J7.2
- net at R2.2: now also J2.4 (Pin_4)
- new net ID: J4.4, R1.2
- no-connect marks 0 -> 2
Other:
- moved on the sheet: R1, R2, R3

Commit message: Worked on sum stuff
Other:
- moved on the sheet: J2, R2, R3
Changed lines of the file:
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@@
 	(paper "A4")
 	(junction
-		(at 67.31 77.47)
+		(at 91.44 74.93)
 		(diameter 0)
 		(color 0 0 0 0)
 	)
 	(no_connect
-		(at 64.77 90.17)
+		(at 88.9 87.63)
 	)
 	(no_connect
@@
 	(wire
 		(pts
-			(xy 62.23 83.82) (xy 62.23 90.17)
+			(xy 86.36 81.28) (xy 86.36 87.63)
 		)
 		(stroke
@@
 	(wire
 		(pts
-			(xy 67.31 64.77) (xy 67.31 68.58)
-		)
-		(stroke
-			(width 0)
-			(type default)
-		)
-	)
-	(wire
-		(pts
-			(xy 67.31 86.36) (xy 67.31 90.17)
-		)
-		(stroke
-			(width 0)
-			(type default)
-		)
-	)
-	(wire
-		(pts
-			(xy 67.31 77.47) (xy 74.93 77.47)
+			(xy 91.44 62.23) (xy 91.44 66.04)
+		)
+		(stroke
+			(width 0)
+			(type default)
+		)
+	)
+	(wire
+		(pts
+			(xy 91.44 83.82) (xy 91.44 87.63)
+		)
+		(stroke
+			(width 0)
+			(type default)
+		)
+	)
+	(wire
+		(pts
+			(xy 91.44 74.93) (xy 99.06 74.93)
 		)
 		(stroke
@@
 	(wire
 		(pts
-			(xy 59.69 85.09) (xy 59.69 90.17)
-		)
-		(stroke
-			(width 0)
-			(type default)
-		)
-	)
-	(wire
-		(pts
-			(xy 67.31 77.47) (xy 67.31 78.74)
+			(xy 83.82 82.55) (xy 83.82 87.63)
+		)
+		(stroke
+			(width 0)
+			(type default)
+		)
+	)
+	(wire
+		(pts
+			(xy 91.44 74.93) (xy 91.44 76.2)
 		)
 		(stroke
@@
 	(wire
 		(pts
-			(xy 67.31 76.2) (xy 67.31 77.47)
+			(xy 91.44 73.66) (xy 91.44 74.93)
 		)
 		(stroke
@@
 	)
 	(label "ADC"
-		(at 74.93 77.47 0)
+		(at 99.06 74.93 0)
 		(effects
 			(font
@@
 	(symbol
 		(lib_id "Device:R")
-		(at 67.31 72.39 0)
+		(at 91.44 69.85 0)
 		(unit 1)
 		(exclude_from_sim no)
@@
 		(fields_autoplaced yes)
 		(property "Reference" "R3"
-			(at 69.85 71.1199 0)
+			(at 93.98 68.5799 0)
 			(effects
 				(font
@@
 		)
 		(property "Value" "R"
-			(at 69.85 73.6599 0)
+			(at 93.98 71.1199 0)
 			(effects
 				(font
@@
 		)
 		(property "Footprint" "Resistor_SMD:R_0805_2012Metric"
-			(at 65.532 72.39 90)
+			(at 89.662 69.85 90)
 			(effects
 				(font
@@
 		)
 		(property "Datasheet" "~"
-			(at 67.31 72.39 0)
+			(at 91.44 69.85 0)
 			(effects
 				(font
@@
 		)
 		(property "Description" "Resistor"
-			(at 67.31 72.39 0)
+			(at 91.44 69.85 0)
 			(effects
 				(font
@@
 	(symbol
 		(lib_id "Connector:Conn_01x04_Pin")
-		(at 62.23 95.25 90)
+		(at 86.36 92.71 90)
 		(unit 1)
 		(exclude_from_sim no)
@@
 		(fields_autoplaced yes)
 		(property "Reference" "J2"
-			(at 63.5 97.79 90)
+			(at 87.63 95.25 90)
 			(effects
 				(font
@@
 		)
 		(property "Value" "Conn_01x04_Pin (MQ series sensor. 4pins (5v, gnd, DO, AO)"
-			(at 63.5 100.33 90)
+			(at 87.63 97.79 90)
 			(effects
 				(font
@@
 		)
 		(property "Footprint" ""
-			(at 62.23 95.25 0)
+			(at 86.36 92.71 0)
 			(effects
 				(font
@@
 		)
 		(property "Datasheet" "~"
-			(at 62.23 95.25 0)
+			(at 86.36 92.71 0)
 			(effects
 				(font
@@
 		)
 		(property "Description" "Generic connector, single row, 01x04, script generated"
-			(at 62.23 95.25 0)
+			(at 86.36 92.71 0)
 			(effects
 				(font
@@
 	(symbol
 		(lib_id "Device:R")
-		(at 67.31 82.55 0)
+		(at 91.44 80.01 0)
 		(unit 1)
 		(exclude_from_sim no)
@@
 		(fields_autoplaced yes)
 		(property "Reference" "R2"
-			(at 69.85 81.2799 0)
+			(at 93.98 78.7399 0)
 			(effects
 				(font
@@
 		)
 		(property "Value" "R"
-			(at 69.85 83.8199 0)
+			(at 93.98 81.2799 0)
 			(effects
 				(font
@@
 		)
 		(property "Footprint" "Resistor_SMD:R_0805_2012Metric"
-			(at 65.532 82.55 90)
+			(at 89.662 80.01 90)
 			(effects
 				(font
@@
 		)
 		(property "Datasheet" "~"
-			(at 67.31 82.55 0)
+			(at 91.44 80.01 0)
 			(effects
 				(font
@@
 		)
 		(property "Description" "Resistor"
-			(at 67.31 82.55 0)
+			(at 91.44 80.01 0)
 			(effects
 				(font
@@
 	(symbol
 		(lib_id "power:GND")
-		(at 67.31 64.77 180)
+		(at 91.44 62.23 180)
 		(unit 1)
 		(exclude_from_sim no)
@@
 		(fields_autoplaced yes)
 		(property "Reference" "#PWR05"
-			(at 67.31 58.42 0)
+			(at 91.44 55.88 0)
 			(effects
 				(font
@@
 		)
 		(property "Value" "GND"
-			(at 67.31 59.69 0)
+			(at 91.44 57.15 0)
 			(effects
 				(font
@@
 		)
 		(property "Footprint" ""
-			(at 67.31 64.77 0)
+			(at 91.44 62.23 0)
 			(effects
 				(font
@@
 		)
 		(property "Datasheet" ""
-			(at 67.31 64.77 0)
+			(at 91.44 62.23 0)
 			(effects
 				(font
@@
 		)
 		(property "Description" "Power symbol creates a global label with name \"GND\" , ground"
-			(at 67.31 64.77 0)
+			(at 91.44 62.23 0)
 			(effects
 				(font
@@
 	(symbol
 		(lib_id "power:+5V")
-		(at 59.69 85.09 90)
+		(at 83.82 82.55 90)
 		(unit 1)
 		(exclude_from_sim no)
@@
 		(fields_autoplaced yes)
 		(property "Reference" "#PWR03"
-			(at 63.5 85.09 0)
+			(at 87.63 82.55 0)
 			(effects
 				(font
@@
 		)
 		(property "Value" "+5V"
-			(at 55.88 85.0899 90)
+			(at 80.01 82.5499 90)
 			(effects
 				(font
@@
 		)
 		(property "Footprint" ""
-			(at 59.69 85.09 0)
+			(at 83.82 82.55 0)
 			(effects
 				(font
@@
 		)
 		(property "Datasheet" ""
-			(at 59.69 85.09 0)
+			(at 83.82 82.55 0)
 			(effects
 				(font
@@
 		)
 		(property "Description" "Power symbol creates a global label with name \"+5V\""
-			(at 59.69 85.09 0)
+			(at 83.82 82.55 0)
 			(effects
 				(font
@@
 	(symbol
 		(lib_id "power:GND")
-		(at 62.23 83.82 180)
+		(at 86.36 81.28 180)
 		(unit 1)
 		(exclude_from_sim no)
@@
 		(fields_autoplaced yes)
 		(property "Reference" "#PWR01"
-			(at 62.23 77.47 0)
+			(at 86.36 74.93 0)
 			(effects
 				(font
@@
 		)
 		(property "Value" "GND"
-			(at 62.23 78.74 0)
+			(at 86.36 76.2 0)
 			(effects
 				(font
@@
 		)
 		(property "Footprint" ""
-			(at 62.23 83.82 0)
+			(at 86.36 81.28 0)
 			(effects
 				(font
@@
 		)
 		(property "Datasheet" ""
-			(at 62.23 83.82 0)
+			(at 86.36 81.28 0)
 			(effects
 				(font
@@
 		)
 		(property "Description" "Power symbol creates a global label with name \"GND\" , ground"
-			(at 62.23 83.82 0)
-			(effects
-				(font
+			(at 86.36 81.28 0)
+			(effects
+				(font
