File: Borealis/sensor-board-temperature/_autosave-sensor-board-temperature.kicad_sch (KiCad schematic)
At the start: 4 parts, among them J2 Conn_01x03_Pin (data connecti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, J5 Conn_01x03_Pin (power connect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

Commit message: Updating changes
Parts:
- removed LTR-390UV-01: ~, batteryholder:SENSOR-SMD_LTR-390UV-01, symbol LTR-390UV-01_2025-12-26-altium-import:root_0_LTR-390UV-01_
Other:
- moved on the sheet: J2, J5, R1
