File: Borealis/sensor-board-IMU/sensor-board-IMU.kicad_sch (KiCad schematic)
At the start: 0 parts

Commit message: stuff
Parts:
- added A1: MPU6050_Module, Charleslabs_Parts:MPU6050_Module, symbol Charleslabs_Parts:MPU6050_Module
- added J1: Conn_01x06_Pin, symbol Connector:Conn_01x06_Pin
- added R1: R, symbol Device:R
Connections:
- new net: J1.6 (Pin_6), R1.2
- new net +3.3V: A1.1 (VCC), J1.2 (Pin_2), R1.1
- new net GND: A1.2 (GND), J1.1 (Pin_1)
- new net SCL: A1.3 (SCL), J1.4 (Pin_4)
- new net SDA: A1.4 (SDA), J1.5 (Pin_5)

Commit message: Updating changes
Parts:
- removed A1: MPU6050_Module, Charleslabs_Parts:MPU6050_Module, symbol Charleslabs_Parts:MPU6050_Module
- removed J1: Conn_01x06_Pin, symbol Connector:Conn_01x06_Pin
- added J2: Conn_01x03_Pin (data connection to main board), batteryholder:1x03 2.3 pitch, symbol Connector:Conn_01x03_Pin
- added J5: Conn_01x03_Pin (power connection to main board), batteryholder:1x03 2.3 pitch, symbol Connector:Conn_01x03_Pin
- added MPU6050: ~, batteryholder:MPU6050-footprint, symbol MPU-6050_C24112_2025-12-25-altium-import:root_0_MPU-6050_C24112_
- R1: footprint (none) -> OptoDevice:R_LDR_4.9x4.2mm_P2.54mm_Vertical
Connections:
- net +3.3V: now also J5.2 (Pin_2), MPU6050.13 (VDD)
- net GND: now also J5.1 (Pin_1), MPU6050.18 (GND)
- net SCL: now also J2.1 (Pin_1), MPU6050.23 (SCL)
- net SDA: now also J2.2 (Pin_2), MPU6050.24 (SDA)
- net ADC: now reaches R1.2
- net ADC: now also J2.3 (Pin_3)
- new net +5V: J5.3 (Pin_3)

Commit message: updated
Parts:
- added C1: 0.1 microf, Capacitor_SMD:CP_Elec_3x5.3, symbol Device:C
- added R2: 10k, Resistor_SMD:R_0805_2012Metric, symbol Device:R
- R1: footprint OptoDevice:R_LDR_4.9x4.2mm_P2.54mm_Vertical -> Resistor_SMD:R_0805_2012Metric
Connections:
- net +3.3V: now also MPU6050.8 (VLOGIC)
- net GND: now also C1.2, R2.1
- net at MPU6050.10 (REGOUT): now also C1.1
- net at MPU6050.11 (FSYNC): now also MPU6050.9 (AD0), R2.2

Commit message: Fixed a few things
Parts:
- removed C1: 0.1 microf, Capacitor_SMD:CP_Elec_3x5.3, symbol Device:C
- removed J2: Conn_01x03_Pin (data connection to main board), batteryholder:1x03 2.3 pitch, symbol Connector:Conn_01x03_Pin
- removed J5: Conn_01x03_Pin (power connection to main board), batteryholder:1x03 2.3 pitch, symbol Connector:Conn_01x03_Pin
- removed MPU6050: ~, batteryholder:MPU6050-footprint, symbol MPU-6050_C24112_2025-12-25-altium-import:root_0_MPU-6050_C24112_
- removed R2: 10k, Resistor_SMD:R_0805_2012Metric, symbol Device:R
- added C5: 100nF, BOREALIS:CAPC17595_95N_KEM, symbol 2026-01-23_05-30-51:C0603C104K5RACTU
- added J4, J7: 878-22-004-10-011101, BOREALIS:8782200410011101, symbol 878-22-004-10-011101:878-22-004-10-011101
- added MPU6500: ~, symbol mm-altium-import:root_0_MPU6500_
Connections:
- net +3.3V: now also C5.2, J4.2, MPU6500.13 (VDD), MPU6500.22 (nCS), MPU6500.8 (VDDIO)
- net +5V: now also J4.3
- net ADC: now also J7.3; no longer R1.2
- net GND: now also C5.1, J4.1, MPU6500.18 (GND), MPU6500.25 (EP), MPU6500.9 (SDO/AD0)
- net SCL: now also J7.1, MPU6500.23 (SCL/SCLK)
- net SDA: now also J7.2, MPU6500.24 (SDA/SDI)
- new net ID: J4.4, R1.2
- no-connect marks 0 -> 1
