File: Borealis/sensor-board-humidity/sensor-board-humidity.kicad_pcb (KiCad board)
At the start: 2 copper layers, 20 x 20 mm, 5 parts, among them J2 Conn_01x03_Pin (data connecti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, J5 Conn_01x03_Pin (power connect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

Commit message: Worked on boards
Parts:
- removed J2: Conn_01x03_Pin (data connection to main board), batteryholder:1x03 2.3 pitch
- removed J5: Conn_01x03_Pin (power connection to main board), batteryholder:1x03 2.3 pitch
- added C5: 100nf, Capacitor_SMD:C_0805_2012Metric, F.Cu at (122.6, 67.3)
- added H1: MountingHole, MountingHole:MountingHole_2.7mm_M2.5_Pad, F.Cu at (119.2, 81.0)
- added R3: 10k, Resistor_SMD:R_0805_2012Metric, F.Cu at (122.9, 72.6)
- added R4: 10k, Resistor_SMD:R_0805_2012Metric, F.Cu at (115.4, 72.5)
- added R5: 10k, Resistor_SMD:R_0805_2012Metric, F.Cu at (119.2, 76.9)
- added U1: MAGNETIC POGO CONN., batteryholder:MAGNETIC POGO CONN., F.Cu at (127.7, 72.1)
- added U2: MAGNETIC POGO CONN., batteryholder:MAGNETIC POGO CONN., F.Cu at (110.7, 72.1)
- SHT31: moved to B.Cu
- moved SHT31 33.9 mm to (119.2, 73.0)
- moved R2 26.6 mm to (119.5, 67.4)
- moved R1 24.1 mm to (116.1, 67.4)
Connections:
- R1 pad 2: /ADC -> /ID
- SHT31 pad 2: GND -> Net-(SHT31-ADDR)
Routing:
- net Net-(SHT31-ADDR): track 0.00 -> 8.95 mm, vias 0 -> 1
- net /SCL: track 6.95 -> 15.8 mm, vias 0 -> 1
- net +3.3V: track 24.4 -> 32.4 mm, vias 0 -> 4
- net /SDA: track 6.62 -> 13.2 mm, vias 0 -> 1
- net /ID: track 0.00 -> 5.50 mm, vias 0 -> 1
- net /ADC: track 5.15 -> 0.00 mm
- net Net-(SHT31-nRESET): track 7.59 -> 3.74 mm, vias 0 -> 1
- net GND: track 5.52 -> 6.47 mm
- added copper zone on F.Cu, net GND
- removed copper zone on B.Cu, net GND
Other:
- board size 20 x 20 mm -> 23.6 x 23.5 mm
- board text added: "Borealis Humidity Sensor"
- board text removed: "Borealis sensor module humidity sensor"
