File: Borealis/sensor-board-humidity/sensor-board-humidity.kicad_sch (KiCad schematic)
At the start: 0 parts

Commit message: stuff
Parts:
- added J1: Conn_01x06_Pin, symbol Connector:Conn_01x06_Pin
- added J2: Conn_01x07_Pin, symbol Connector:Conn_01x07_Pin
- added R1: R, symbol Device:R
Connections:
- new net: J1.6 (Pin_6), R1.2
- new net +3.3V: J1.2 (Pin_2), R1.1
- new net GND: J1.1 (Pin_1)

Commit message: Updating changes
Parts:
- removed J1: Conn_01x06_Pin, symbol Connector:Conn_01x06_Pin
- removed J2: Conn_01x07_Pin, symbol Connector:Conn_01x07_Pin
- added J2: Conn_01x03_Pin (data connection to main board), batteryholder:1x03 2.3 pitch, symbol Connector:Conn_01x03_Pin
- added J5: Conn_01x03_Pin (power connection to main board), batteryholder:1x03 2.3 pitch, symbol Connector:Conn_01x03_Pin
- added SHT31: ~, batteryholder:sht31-footprint, symbol SHT31-DIS-F2.5KS_2025-12-25-altium-import:root_0_SHT31-DIS-F2.5KS_
- R1: footprint (none) -> OptoDevice:R_LDR_4.9x4.2mm_P2.54mm_Vertical
Connections:
- net +3.3V: now also J5.2 (Pin_2), SHT31.5 (VDD)
- net GND: now also J5.1 (Pin_1), SHT31.8 (VSS)
- net ADC: now reaches R1.2
- net ADC: now also J2.3 (Pin_3)
- new net +5V: J5.3 (Pin_3)
- new net SCL: J2.1 (Pin_1), SHT31.4 (SCL)
- new net SDA: J2.2 (Pin_2), SHT31.1 (SDA)

Commit message: updated
Parts:
- added R2: 10k, Resistor_SMD:R_0805_2012Metric, symbol Device:R
- R1: footprint OptoDevice:R_LDR_4.9x4.2mm_P2.54mm_Vertical -> Resistor_SMD:R_0805_2012Metric
Connections:
- net +3.3V: now also R2.2
- net GND: now also SHT31.2 (ADDR), SHT31.7 (R), SHT31.9 (EP)
- net at SHT31.6 (nRESET): now also R2.1

Commit message: Fixed a few things
Parts:
- removed J2: Conn_01x03_Pin (data connection to main board), batteryholder:1x03 2.3 pitch, symbol Connector:Conn_01x03_Pin
- removed J5: Conn_01x03_Pin (power connection to main board), batteryholder:1x03 2.3 pitch, symbol Connector:Conn_01x03_Pin
- added C5: C0603C104K5RACTU, BOREALIS:CAPC17595_95N_KEM, symbol 2026-01-23_05-30-51:C0603C104K5RACTU
- added J4, J7: 878-22-004-10-011101, BOREALIS:8782200410011101, symbol 878-22-004-10-011101:878-22-004-10-011101
Connections:
- net +3.3V: now also C5.1, J4.2
- net +5V: now also J4.3
- net ADC: now also J7.3; no longer R1.2
- net GND: now also C5.2, J4.1
- net SCL: now also J7.1
- net SDA: now also J7.2
- new net ID: J4.4, R1.2
- no-connect marks 0 -> 1
Other:
- moved on the sheet: R2, SHT31

Commit message: Worked on boards
Parts:
- removed J4, J7: 878-22-004-10-011101, BOREALIS:8782200410011101, symbol 878-22-004-10-011101:878-22-004-10-011101
- added H1: MountingHole, MountingHole:MountingHole_2.7mm_M2.5_Pad, symbol Mechanical:MountingHole
- added R3, R4, R5: 10k, Resistor_SMD:R_0805_2012Metric, symbol Device:R
- added U1, U2: MAGNETIC POGO CONN., batteryholder:MAGNETIC POGO CONN., symbol magnetic_pogo_conn.:MAGNETIC_POGO_CONN.
- C5: value C0603C104K5RACTU -> 100nf; footprint BOREALIS:CAPC17595_95N_KEM -> Capacitor_SMD:C_0805_2012Metric
Connections:
- net +3.3V: now also R4.1, R5.2, U2.2
- net +5V: now also U2.3
- net ADC: now also U1.2
- net GND: now also R3.1, U2.1; no longer SHT31.2 (ADDR)
- net ID: now also U2.4
- net SCL: now also R4.2, U1.4
- net SDA: now also R5.1, U1.3
- new net: R3.2, SHT31.2 (ADDR)
- no-connect marks 1 -> 2
