File: Borealis/sensor-board-light/sensor-board-light.kicad_pcb (KiCad board)
At the start: 2 copper layers, 31.5 x 20 mm, 6 parts, among them J1 Conn_01x04_Pin, J2 Conn_01x03_Pin (data connecti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, J3 Conn_01x04_Pin, J5 Conn_01x03_Pin (power connect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

Commit message: Worked on sum stuff
Other:
- outline, holes or cut-outs redrawn
Changed lines of the file:
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@@
+	)
+	(gr_circle
+		(center 112.35 73)
+		(end 113.5 73)
+		(stroke
+			(width 0.05)
+			(type solid)
+		)
+		(fill no)
+		(layer "Edge.Cuts")
 	)
 	(gr_circle
@@
 		(stroke
 			(width 0.05)
+			(type solid)
+		)
+		(fill no)
+		(layer "Edge.Cuts")
+	)
+	(gr_circle
+		(center 111.85 83)
+		(end 113 83)
+		(stroke
+			(width 0.05)

Commit message: Worked on boards
Parts:
- removed J2: Conn_01x03_Pin (data connection to main board), batteryholder:1x03 2.3 pitch
- removed J5: Conn_01x03_Pin (power connection to main board), batteryholder:1x03 2.3 pitch
- added C1: 100nF, Capacitor_SMD:C_0805_2012Metric, F.Cu at (137.4, 90.8)
- added H1: MountingHole, MountingHole:MountingHole_2.7mm_M2.5_Pad, F.Cu at (142.3, 79.4)
- added H2: MountingHole, MountingHole:MountingHole_2.7mm_M2.5_Pad, F.Cu at (126.2, 88.1)
- added H3: MountingHole, MountingHole:MountingHole_2.7mm_M2.5_Pad, F.Cu at (126.2, 93.9)
- added R3: 10k, Resistor_SMD:R_0805_2012Metric, F.Cu at (133.7, 94.2)
- added R5: 10k, Resistor_SMD:R_0805_2012Metric, F.Cu at (145.1, 74.0)
- added R6: 10k, Resistor_SMD:R_0805_2012Metric, F.Cu at (139.8, 73.9)
- added U1: MAGNETIC POGO CONN., batteryholder:MAGNETIC POGO CONN., F.Cu at (150.8, 70.6)
- added U2: MAGNETIC POGO CONN., batteryholder:MAGNETIC POGO CONN., F.Cu at (133.8, 70.6)
- J1: footprint Connector_PinHeader_2.54mm:PinHeader_1x04_P2.54mm_Vertical -> Connector_JST:JST_PH_B4B-PH-K_1x04_P2.00mm_Vertical; moved to B.Cu
- moved J3 36.7 mm to (141.3, 87.2)
- moved LTR-390UV-01 25.1 mm to (133.7, 90.6), turned to 90 degrees
- moved J1 16.2 mm to (145.4, 69.1), turned to 180 degrees
- moved R1 12.1 mm to (139.2, 65.1), turned to 180 degrees
Connections:
- LTR-390UV-01 pad 5: unconnected-(LTR-390UV-01-INT-Pad5) -> Net-(LTR-390UV-01-INT)
- R1 pad 2: /ADC -> /ID
Routing:
- net /3.3v: track 6.09 -> 22.7 mm
- net +3.3V: track 12.9 -> 23.8 mm
- net /SCL: track 9.23 -> 17.8 mm, vias 0 -> 1
- net Net-(LTR-390UV-01-INT): track 0.00 -> 7.63 mm
- net /SCL1: track 5.61 -> 12.3 mm
- net /SDA: track 9.33 -> 14.7 mm, vias 0 -> 1
- net /ID: track 0.00 -> 4.54 mm
- net /ADC: track 4.27 -> 0.00 mm
- net /SDA1: track 6.45 -> 9.02 mm
- net GND: track 24.7 -> 23.9 mm
Other:
- board size 31.5 x 20 mm -> 30.9 x 38 mm
- board text added: "Borealis Light Sensor"
- board text added: "External light sensor module"
- board text removed: "Borealis sensor module Magnetometer"
