File: Borealis/sensor-board-light/sensor-board-light.kicad_sch (KiCad schematic)
At the start: 4 parts, among them J2 Conn_01x03_Pin (data connecti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, J5 Conn_01x03_Pin (power connect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

Commit message: .
Parts:
- added J1, J3: Conn_01x04_Pin, Connector_PinHeader_2.54mm:PinHeader_1x04_P2.54mm_Vertical, symbol Connector:Conn_01x04_Pin
- J2, J5: footprint (none) -> batteryholder:1x03 2.3 pitch
- R1: footprint OptoDevice:R_LDR_4.9x4.2mm_P2.54mm_Vertical -> Resistor_SMD:R_0805_2012Metric
Connections:
- net +3.3V: now also J1.2 (Pin_2), J3.2 (Pin_2)
- net GND: now also J1.1 (Pin_1), J3.1 (Pin_1)
- net SCL: now also J1.4 (Pin_4), J3.4 (Pin_4)
- net SDA: now also J1.3 (Pin_3), J3.3 (Pin_3)

Commit message: updated
Connections:
- net +3.3V: no longer J3.2 (Pin_2), LTR-390UV-01.1 (VDD)
- net SCL: no longer J3.4 (Pin_4), LTR-390UV-01.4 (SCL)
- net SDA: no longer J3.3 (Pin_3), LTR-390UV-01.6 (SDA)
- new net 3.3v: J3.2 (Pin_2), LTR-390UV-01.1 (VDD)
- new net SCL1: J3.4 (Pin_4), LTR-390UV-01.4 (SCL)
- new net SDA1: J3.3 (Pin_3), LTR-390UV-01.6 (SDA)

Commit message: Fixed a few things
Parts:
- removed J2: Conn_01x03_Pin (data connection to main board), batteryholder:1x03 2.3 pitch, symbol Connector:Conn_01x03_Pin
- removed J5: Conn_01x03_Pin (power connection to main board), batteryholder:1x03 2.3 pitch, symbol Connector:Conn_01x03_Pin
- added C5: 100nF, BOREALIS:CAPC17595_95N_KEM, symbol 2026-01-23_05-30-51:C0603C104K5RACTU
- added J4, J7: 878-22-004-10-011101, BOREALIS:8782200410011101, symbol 878-22-004-10-011101:878-22-004-10-011101
- added R2, R3, R4: 10k, Resistor_SMD:R_0805_2012Metric, symbol Device:R
Connections:
- net +3.3V: now also C5.2, J4.2
- net +5V: now also J4.3
- net 3.3v: now also R2.1, R3.1, R4.1
- net ADC: now also J7.3; no longer R1.2
- net GND: now also C5.1, J4.1
- net SCL: now also J7.1
- net SCL1: now also R4.2
- net SDA: now also J7.2
- net SDA1: now also R2.2
- net at LTR-390UV-01.5 (INT): now also R3.2
- new net ID: J4.4, R1.2
- no-connect marks 0 -> 1
Other:
- note added: "External Module"
- moved on the sheet: J1, J3, LTR-390UV-01

Commit message: Worked on boards
Parts:
- removed C5: 100nF, BOREALIS:CAPC17595_95N_KEM, symbol 2026-01-23_05-30-51:C0603C104K5RACTU
- removed J4, J7: 878-22-004-10-011101, BOREALIS:8782200410011101, symbol 878-22-004-10-011101:878-22-004-10-011101
- removed R2, R4: 10k, Resistor_SMD:R_0805_2012Metric, symbol Device:R
- added C1: 100nF, Capacitor_SMD:C_0805_2012Metric, symbol 2026-01-23_05-30-51:C0603C104K5RACTU
- added H1, H2, H3: MountingHole, MountingHole:MountingHole_2.7mm_M2.5_Pad, symbol Mechanical:MountingHole
- added R5, R6: 10k, Resistor_SMD:R_0805_2012Metric, symbol Device:R
- added U2, U3: MAGNETIC POGO CONN., batteryholder:MAGNETIC POGO CONN., symbol magnetic_pogo_conn.:MAGNETIC_POGO_CONN.
- J1: footprint Connector_PinHeader_2.54mm:PinHeader_1x04_P2.54mm_Vertical -> Connector_JST:JST_PH_B4B-PH-K_1x04_P2.00mm_Vertical
Connections:
- net +3.3V: now also R5.1, R6.1, U3.2
- net +5V: now also U3.3
- net 3.3v: now also C1.2
- net ADC: now also U2.2
- net GND: now also C1.1, U3.1
- net ID: now also U3.4
- net SCL: now also R6.2, U2.4
- net SDA: now also R5.2, U2.3
- no-connect marks 1 -> 2
