File: Borealis/sensor-board-magnetic-field/sensor-board-magnetic-field.kicad_pcb (KiCad board)
At the start: 2 copper layers, 35 x 30 mm, 4 parts, among them J2 Conn_01x03_Pin (data connecti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, J5 Conn_01x03_Pin (power connect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

Commit message: updated
Parts:
- removed MPU9250: ~, batteryholder:MPU9250
- added TLV493D1: ~, batteryholder:TLV493D, F.Cu at (93.2, 118.1)
- moved J5 39.0 mm to (90.9, 126.0), turned to 0 degrees
- moved R1 13.3 mm to (99.0, 118.1)
- moved J2 4.56 mm to (90.4, 111.0), turned to 0 degrees
Routing:
- net +3.3V: track 0.00 -> 12.2 mm
- net GND: track 0.00 -> 10.8 mm
- net /ADC: track 0.00 -> 7.71 mm
- net /SDA: track 0.00 -> 6.74 mm
- net /SCL: track 0.00 -> 6.71 mm
Other:
- board size 35 x 30 mm -> 20 x 20 mm
- board text added: "Borealis sensor module Magnetometer"
- board text removed: "Borealis sensor board 9-axis IMU"

Commit message: Worked on boards
Parts:
- removed J2: Conn_01x03_Pin (data connection to main board), batteryholder:1x03 2.3 pitch
- removed J5: Conn_01x03_Pin (power connection to main board), batteryholder:1x03 2.3 pitch
- added C5: 100nF, Capacitor_SMD:C_0805_2012Metric, F.Cu at (120.8, 96.9)
- added H1: MountingHole, MountingHole:MountingHole_2.7mm_M2.5_Pad, F.Cu at (118.9, 111.1)
- added R2: 10K, Resistor_SMD:R_0805_2012Metric, F.Cu at (120.3, 104.6)
- added R3: 10K, Resistor_SMD:R_0805_2012Metric, F.Cu at (116.7, 104.7)
- added U1: MAGNETIC POGO CONN., batteryholder:MAGNETIC POGO CONN., F.Cu at (127.4, 102.3)
- added U2: MAGNETIC POGO CONN., batteryholder:MAGNETIC POGO CONN., F.Cu at (110.4, 102.3)
- TLV493D1: moved to B.Cu
- moved TLV493D1 31.3 mm to (118.9, 100.3)
- moved R1 27.2 mm to (116.2, 97.0), turned to 180 degrees
Connections:
- R1 pad 2: /ADC -> /ID
Routing:
- net GND: track 10.8 -> 24.5 mm, vias 0 -> 1
- net +3.3V: track 12.2 -> 24.9 mm, vias 0 -> 4
- net /SCL: track 6.71 -> 15.2 mm, vias 0 -> 1
- net /ADC: track 7.71 -> 0.00 mm
- net /ID: track 0.00 -> 4.86 mm
- net /SDA: track 6.74 -> 9.83 mm, vias 0 -> 1
Other:
- board size 20 x 20 mm -> 23.6 x 23.5 mm
- board text added: "Borealis Magnetometer"
- board text removed: "Borealis sensor module Magnetometer"
