File: Borealis/sensor-board-magnetic-field/sensor-board-magnetic-field.kicad_sch (KiCad schematic)
At the start: 0 parts

Commit message: Updating changes
Parts:
- added J2: Conn_01x03_Pin (data connection to main board), batteryholder:1x03 2.3 pitch, symbol Connector:Conn_01x03_Pin
- added J5: Conn_01x03_Pin (power connection to main board), batteryholder:1x03 2.3 pitch, symbol Connector:Conn_01x03_Pin
- added MPU9250: ~, batteryholder:MPU9250, symbol MPU9250_2025-12-26-altium-import:root_0_MPU9250_
- added R1: R, Resistor_SMD:R_0805_2012Metric, symbol Device:R
Connections:
- new net +3.3V: J5.2 (Pin_2), MPU9250.1 (VCC), R1.1
- new net +5V: J5.3 (Pin_3)
- new net ADC: J2.3 (Pin_3), R1.2
- new net GND: J5.1 (Pin_1), MPU9250.2 (GND)
- new net SCL: J2.1 (Pin_1), MPU9250.3 (SCL)
- new net SDA: J2.2 (Pin_2), MPU9250.4 (SDA)
- no-connect marks 0 -> 7

Commit message: .
Parts:
- removed MPU9250: ~, batteryholder:MPU9250, symbol MPU9250_2025-12-26-altium-import:root_0_MPU9250_
- added TLV493D1: ~, batteryholder:TLV493D, symbol TLV493DA1B6HTSA2_2025-12-27-altium-import:root_0_TLV493DA1B6HTSA2_
Connections:
- net +3.3V: now also TLV493D1.4 (VDD)
- net GND: now also TLV493D1.2 (GND), TLV493D1.3 (GND), TLV493D1.5 (GND)
- net SCL: now also TLV493D1.1 (SCL/INT)
- net SDA: now also TLV493D1.6 (SDA/ADDR)
- no-connect marks 7 -> 1

Commit message: Fixed a few things
Parts:
- removed J2: Conn_01x03_Pin (data connection to main board), batteryholder:1x03 2.3 pitch, symbol Connector:Conn_01x03_Pin
- removed J5: Conn_01x03_Pin (power connection to main board), batteryholder:1x03 2.3 pitch, symbol Connector:Conn_01x03_Pin
- added C5: 100nF, BOREALIS:CAPC17595_95N_KEM, symbol 2026-01-23_05-30-51:C0603C104K5RACTU
- added J4, J7: 878-22-004-10-011101, BOREALIS:8782200410011101, symbol 878-22-004-10-011101:878-22-004-10-011101
- added R2, R3: 10K, Resistor_SMD:R_0805_2012Metric, symbol Device:R
Connections:
- net +3.3V: now also C5.2, J4.2, R2.1, R3.1
- net +5V: now also J4.3
- net ADC: now also J7.3; no longer R1.2
- net GND: now also C5.1, J4.1
- net SCL: now also J7.1, R3.2
- net SDA: now also J7.2, R2.2
- new net ID: J4.4, R1.2

Commit message: Worked on boards
Parts:
- removed J4, J7: 878-22-004-10-011101, BOREALIS:8782200410011101, symbol 878-22-004-10-011101:878-22-004-10-011101
- added H1: MountingHole, MountingHole:MountingHole_2.7mm_M2.5_Pad, symbol Mechanical:MountingHole
- added U2, U3: MAGNETIC POGO CONN., batteryholder:MAGNETIC POGO CONN., symbol magnetic_pogo_conn.:MAGNETIC_POGO_CONN.
- C5: footprint BOREALIS:CAPC17595_95N_KEM -> Capacitor_SMD:C_0805_2012Metric
Connections:
- net +3.3V: now also U3.2
- net +5V: now also U3.3
- net ADC: now also U2.2
- net GND: now also U3.1
- net ID: now also U3.4
- net SCL: now also U2.4
- net SDA: now also U2.3
