File: Borealis/sensor-board-pressure/sensor-board-pressure.kicad_sch (KiCad schematic)
At the start: 0 parts

Commit message: Added sensor board
Parts:
- added J1: Conn_01x06_Pin, Connector_PinHeader_2.54mm:PinHeader_1x06_P2.54mm_Vertical, symbol Connector:Conn_01x06_Pin
- added J2: Conn_01x08_Pin (BMP390), Adafruit BMP390:1X08_ROUND_70, symbol Connector:Conn_01x08_Pin
- added R1: R, OptoDevice:R_LDR_4.9x4.2mm_P2.54mm_Vertical, symbol Device:R
Connections:
- new net: J1.6 (Pin_6), R1.2
- new net +3.3V: J1.2 (Pin_2), J2.1 (Pin_1), R1.1
- new net GND: J1.1 (Pin_1), J2.3 (Pin_3)
- new net SCL: J1.4 (Pin_4), J2.4 (Pin_4)
- new net SDA: J1.5 (Pin_5), J2.6 (Pin_6)

Commit message: Updating changes
Parts:
- removed J1: Conn_01x06_Pin, Connector_PinHeader_2.54mm:PinHeader_1x06_P2.54mm_Vertical, symbol Connector:Conn_01x06_Pin
- removed J2: Conn_01x08_Pin (BMP390), Adafruit BMP390:1X08_ROUND_70, symbol Connector:Conn_01x08_Pin
- added BMP390: ~, Adafruit BMP390:BMP388, symbol BMP390_2025-12-25-altium-import:root_0_BMP390_
- added J2: Conn_01x03_Pin (data connection to main board), batteryholder:1x03 2.3 pitch, symbol Connector:Conn_01x03_Pin
- added J5: Conn_01x03_Pin (power connection to main board), batteryholder:1x03 2.3 pitch, symbol Connector:Conn_01x03_Pin
Connections:
- net +3.3V: now also BMP390.1 (VDDIO), BMP390.10 (VDD), BMP390.6 (CSB), J5.2 (Pin_2)
- net GND: now also BMP390.5 (SDO), BMP390.8 (VSS), J5.1 (Pin_1)
- net SCL: now also BMP390.2 (SCK), J2.1 (Pin_1)
- net SDA: now also BMP390.4 (SDI), J2.2 (Pin_2)
- net ADC: now reaches R1.2
- net ADC: now also J2.3 (Pin_3)
- new net +5V: J5.3 (Pin_3)

Commit message: Added barometric sensor board
Parts:
- R1: footprint OptoDevice:R_LDR_4.9x4.2mm_P2.54mm_Vertical -> Resistor_SMD:R_0805_2012Metric
Changed lines of the file:
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@@
 			)
 		)
-		(property "Footprint" "OptoDevice:R_LDR_4.9x4.2mm_P2.54mm_Vertical"
+		(property "Footprint" "Resistor_SMD:R_0805_2012Metric"
 			(at 90.932 106.68 90)
 			(effects

Commit message: updated
Parts:
- added R2: 10k, Resistor_SMD:R_0805_2012Metric, symbol Device:R
Connections:
- net +3.3V: now also R2.1; no longer BMP390.6 (CSB)
- net GND: now also BMP390.3 (VSS), BMP390.9 (VSS)
- new net: BMP390.6 (CSB), R2.2
Changed lines of the file:
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@@
 	(generator_version "9.0")
 	(paper "A4")
+	(junction
+		(at 73.66 83.82)
+		(diameter 0)
+		(color 0 0 0 0)
+	)
 	(wire
 		(pts
@@
 	(wire
 		(pts
+			(xy 44.45 83.82) (xy 50.8 83.82)
+		)
+		(stroke
+			(width 0)
+			(type default)
+		)
+	)
+	(wire
+		(pts
+			(xy 77.47 97.79) (xy 77.47 100.33)
+		)
+		(stroke
+			(width 0)
+			(type default)
+		)
+	)
+	(wire
+		(pts
 			(xy 96.52 59.69) (xy 101.6 59.69)
 		)
@@
 	(wire
 		(pts
+			(xy 77.47 88.9) (xy 77.47 90.17)
+		)
+		(stroke
+			(width 0)
+			(type default)
+		)
+	)
+	(wire
+		(pts
 			(xy 46.99 81.28) (xy 50.8 81.28)
 		)
@@
 		(pts
 			(xy 46.99 86.36) (xy 50.8 86.36)
+		)
+		(stroke
+			(width 0)
+			(type default)
+		)
+	)
+	(wire
+		(pts
+			(xy 73.66 81.28) (xy 73.66 83.82)
 		)
 		(stroke
@@
 	)
 	(symbol
+		(lib_id "power:GND")
+		(at 44.45 83.82 270)
+		(unit 1)
+		(exclude_from_sim no)
+		(in_bom yes)
+		(on_board yes)
+		(dnp no)
+		(fields_autoplaced yes)
+		(property "Reference" "#PWR05"
+			(at 38.1 83.82 0)
+			(effects
+				(font
+					(size 1.27 1.27)
+				)
+				(hide yes)
+			)
+		)
+		(property "Value" "GND"
+			(at 40.64 83.8199 90)
+			(effects
+				(font
+					(size 1.27 1.27)
+				)
+				(justify right)
+			)
+		)
+		(property "Footprint" ""
+			(at 44.45 83.82 0)
+			(effects
+				(font
+					(size 1.27 1.27)
+				)
+				(hide yes)
+			)
+		)
+		(property "Datasheet" ""
+			(at 44.45 83.82 0)
+			(effects
+				(font
+					(size 1.27 1.27)
+				)
+				(hide yes)
+			)
+		)
+		(property "Description" "Power symbol creates a global label with name \"GND\" , ground"
+			(at 44.45 83.82 0)
+			(effects
+				(font
+					(size 1.27 1.27)
+				)
+				(hide yes)
+			)
+		)
+		(pin "1"
+		)
+		(instances
+			(project ""
+				(path "/073ec1fb-7e7a-4821-a0d2-1e02de7627d5"
+					(reference "#PWR05")
+					(unit 1)
+				)
+			)
+		)
+	)
+	(symbol
 		(lib_id "BMP390_2025-12-25-altium-import:root_0_BMP390_")
 		(at 62.23 83.82 0)
@@
 	)
 	(symbol
+		(lib_id "power:+3.3V")
+		(at 77.47 100.33 180)
+		(unit 1)
+		(exclude_from_sim no)
+		(in_bom yes)
+		(on_board yes)
+		(dnp no)
+		(fields_autoplaced yes)
+		(property "Reference" "#PWR07"
+			(at 77.47 96.52 0)
+			(effects
+				(font
+					(size 1.27 1.27)
+				)
+				(hide yes)
+			)
+		)
+		(property "Value" "+3.3V"
+			(at 77.47 105.41 0)
+			(effects
+				(font
+					(size 1.27 1.27)
+				)
+			)
+		)
+		(property "Footprint" ""
+			(at 77.47 100.33 0)
+			(effects
+				(font
+					(size 1.27 1.27)
+				)
+				(hide yes)
+			)
+		)
+		(property "Datasheet" ""
+			(at 77.47 100.33 0)
+			(effects
+				(font
+					(size 1.27 1.27)
+				)
+				(hide yes)
+			)
+		)
+		(property "Description" "Power symbol creates a global label with name \"+3.3V\""
+			(at 77.47 100.33 0)
+			(effects
+				(font
+					(size 1.27 1.27)
+				)
+				(hide yes)
+			)
+		)
+		(pin "1"
+		)
+		(instances
+			(project ""
+				(path "/073ec1fb-7e7a-4821-a0d2-1e02de7627d5"
+					(reference "#PWR07")
+					(unit 1)
+				)
+			)
+		)
+	)
+	(symbol
 		(lib_id "power:GND")
 		(at 99.06 80.01 270)
@@
 	)
 	(symbol
+		(lib_id "Device:R")
+		(at 77.47 93.98 180)
+		(unit 1)
+		(exclude_from_sim no)
+		(in_bom yes)
+		(on_board yes)
+		(dnp no)
+		(fields_autoplaced yes)
+		(property "Reference" "R2"
+			(at 80.01 92.7099 0)
+			(effects
+				(font
+					(size 1.27 1.27)
+				)
+				(justify right)
+			)
+		)
+		(property "Value" "10k"
+			(at 80.01 95.2499 0)
+			(effects
+				(font
+					(size 1.27 1.27)
+				)
+				(justify right)
+			)
+		)
+		(property "Footprint" "Resistor_SMD:R_0805_2012Metric"
+			(at 79.248 93.98 90)
+			(effects
+				(font
+					(size 1.27 1.27)
+				)
+				(hide yes)
+			)
+		)
+		(property "Datasheet" "~"
+			(at 77.47 93.98 0)
+			(effects
+				(font
+					(size 1.27 1.27)
+				)
+				(hide yes)
+			)
+		)
+		(property "Description" "Resistor"
+			(at 77.47 93.98 0)
+			(effects
+				(font
+					(size 1.27 1.27)
+				)
+				(hide yes)
+			)
+		)
+		(pin "2"
+		)
+		(pin "1"
+		)
+		(instances
+			(project ""
+				(path "/073ec1fb-7e7a-4821-a0d2-1e02de7627d5"
+					(reference "R2")
+					(unit 1)
+				)
+			)
+		)
+	)
+	(symbol
 		(lib_id "power:GND")
 		(at 48.26 88.9 270)
@@
 					(unit 1)
 				)
-			)
-		)
-	)
-	(symbol
-		(lib_id "power:+3.3V")
-		(at 77.47 88.9 270)
-		(unit 1)
-		(exclude_from_sim no)
-		(in_bom yes)
-		(on_board yes)
-		(dnp no)
-		(fields_autoplaced yes)
-		(property "Reference" "#PWR05"
-			(at 73.66 88.9 0)
-			(effects
-				(font
-					(size 1.27 1.27)
-				)
-				(hide yes)
-			)
-		)
-		(property "Value" "+3.3V"
-			(at 81.28 88.8999 90)
-			(effects
-				(font
-					(size 1.27 1.27)
-				)
-				(justify left)
-			)
-		)
-		(property "Footprint" ""
-			(at 77.47 88.9 0)
-			(effects
-				(font
-					(size 1.27 1.27)
-				)
-				(hide yes)
-			)
-		)
-		(property "Datasheet" ""
-			(at 77.47 88.9 0)
-			(effects
-				(font
-					(size 1.27 1.27)
-				)
-				(hide yes)
-			)
-		)
-		(property "Description" "Power symbol creates a global label with name \"+3.3V\""
-			(at 77.47 88.9 0)
-			(effects
-				(font
-					(size 1.27 1.27)
-				)
-				(hide yes)
-			)
-		)
-		(pin "1"
-		)
-		(instances
-			(project ""
-				(path "/073ec1fb-7e7a-4821-a0d2-1e02de7627d5"
-					(reference "#PWR05")
-					(unit 1)
-				)

Commit message: Fixed a few things
Parts:
- removed J2: Conn_01x03_Pin (data connection to main board), batteryholder:1x03 2.3 pitch, symbol Connector:Conn_01x03_Pin
- removed J5: Conn_01x03_Pin (power connection to main board), batteryholder:1x03 2.3 pitch, symbol Connector:Conn_01x03_Pin
- added C1, C5: 100nF, BOREALIS:CAPC17595_95N_KEM, symbol 2026-01-23_05-30-51:C0603C104K5RACTU
- added J4, J7: 878-22-004-10-011101, BOREALIS:8782200410011101, symbol 878-22-004-10-011101:878-22-004-10-011101
- added R3: 4.7kOhms, Resistor_SMD:R_0805_2012Metric, symbol Device:R
- R2: value 10k -> 4.7kOhms
Connections:
- net +3.3V: now also BMP390.6 (CSB), R2.2, C1.2, C5.2, J4.2, R3.2; no longer R2.1
- net +5V: now also J4.3
- net ADC: now also J7.3; no longer R1.2
- net GND: now also C1.1, C5.1, J4.1
- net SCL: now also J7.1, R3.1
- net SDA: now also R2.1, J7.2
- new net ID: J4.4, R1.2
- no-connect marks 0 -> 1

Commit message: Worked on sum stuff
Parts:
- removed J4, J7: 878-22-004-10-011101, BOREALIS:8782200410011101, symbol 878-22-004-10-011101:878-22-004-10-011101
- added U1, U2: MAGNETIC POGO CONN., batteryholder:MAGNETIC POGO CONN., symbol magnetic_pogo_conn.:MAGNETIC_POGO_CONN.
- C1, C5: footprint BOREALIS:CAPC17595_95N_KEM -> Capacitor_SMD:C_0805_2012Metric
Connections:
- net +3.3V: now also U2.2
- net +5V: now also U2.3
- net ADC: now also U1.2
- net GND: now also U2.1
- net ID: now also U2.4
- net SCL: now also U1.4
- net SDA: now also U1.3
- no-connect marks 1 -> 2

Commit message: Worked on boards
Parts:
- added H1: MountingHole, MountingHole:MountingHole_2.7mm_M2.5_Pad, symbol Mechanical:MountingHole
Other:
- moved on the sheet: C1
Changed lines of the file:
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@@
+	)
+	(junction
+		(at 41.91 68.58)
+		(diameter 0)
+		(color 0 0 0 0)
 	)
 	(junction
@@
 	)
 	(junction
-		(at 22.86 83.82)
+		(at 41.91 83.82)
 		(diameter 0)
 		(color 0 0 0 0)
@@
 	(wire
 		(pts
+			(xy 41.91 78.74) (xy 41.91 83.82)
+		)
+		(stroke
+			(width 0)
+			(type default)
+		)
+	)
+	(wire
+		(pts
 			(xy 77.47 78.74) (xy 77.47 73.66)
 		)
@@
 	(wire
 		(pts
-			(xy 20.32 83.82) (xy 22.86 83.82)
+			(xy 20.32 83.82) (xy 41.91 83.82)
 		)
 		(stroke
@@
 	(wire
 		(pts
+			(xy 45.72 68.58) (xy 41.91 68.58)
+		)
+		(stroke
+			(width 0)
+			(type default)
+		)
+	)
+	(wire
+		(pts
 			(xy 48.26 88.9) (xy 50.8 88.9)
 		)
@@
 	(wire
 		(pts
+			(xy 41.91 83.82) (xy 50.8 83.82)
+		)
+		(stroke
+			(width 0)
+			(type default)
+		)
+	)
+	(wire
+		(pts
 			(xy 17.78 81.28) (xy 22.86 81.28)
 		)
@@
 	(wire
 		(pts
+			(xy 41.91 68.58) (xy 41.91 71.12)
+		)
+		(stroke
+			(width 0)
+			(type default)
+		)
+	)
+	(wire
+		(pts
 			(xy 73.66 78.74) (xy 77.47 78.74)
 		)
@@
 	(wire
 		(pts
+			(xy 41.91 63.5) (xy 41.91 68.58)
+		)
+		(stroke
+			(width 0)
+			(type default)
+		)
+	)
+	(wire
+		(pts
 			(xy 73.66 83.82) (xy 86.36 83.82)
 		)
@@
 	(wire
 		(pts
-			(xy 22.86 83.82) (xy 50.8 83.82)
-		)
-		(stroke
-			(width 0)
-			(type default)
-		)
-	)
-	(wire
-		(pts
 			(xy 127 55.88) (xy 120.65 55.88)
 		)
@@
 		(pts
 			(xy 31.75 86.36) (xy 38.1 86.36)
+		)
+		(stroke
+			(width 0)
+			(type default)
+		)
+	)
+	(wire
+		(pts
+			(xy 45.72 78.74) (xy 45.72 68.58)
 		)
 		(stroke
@@
 	(symbol
 		(lib_id "power:+3.3V")
-		(at 45.72 78.74 90)
-		(unit 1)
-		(exclude_from_sim no)
-		(in_bom yes)
-		(on_board yes)
-		(dnp no)
-		(fields_autoplaced yes)
-		(property "Reference" "#PWR04"
-			(at 49.53 78.74 0)
-			(effects
-				(font
-					(size 1.27 1.27)
-				)
-				(hide yes)
-			)
-		)
-		(property "Value" "+3.3V"
-			(at 41.91 78.7399 90)
-			(effects
-				(font
-					(size 1.27 1.27)
-				)
-				(justify left)
-			)
-		)
-		(property "Footprint" ""
-			(at 45.72 78.74 0)
-			(effects
-				(font
-					(size 1.27 1.27)
-				)
-				(hide yes)
-			)
-		)
-		(property "Datasheet" ""
-			(at 45.72 78.74 0)
-			(effects
-				(font
-					(size 1.27 1.27)
-				)
-				(hide yes)
-			)
-		)
-		(property "Description" "Power symbol creates a global label with name \"+3.3V\""
-			(at 45.72 78.74 0)
-			(effects
-				(font
-					(size 1.27 1.27)
-				)
-				(hide yes)
-			)
-		)
-		(pin "1"
-		)
-		(instances
-			(project ""
-				(path "/073ec1fb-7e7a-4821-a0d2-1e02de7627d5"
-					(reference "#PWR04")
-					(unit 1)
-				)
-			)
-		)
-	)
-	(symbol
-		(lib_id "power:+3.3V")
-		(at 22.86 91.44 180)
+		(at 41.91 63.5 0)
 		(unit 1)
 		(exclude_from_sim no)
@@
 		(fields_autoplaced yes)
 		(property "Reference" "#PWR09"
-			(at 22.86 87.63 0)
+			(at 41.91 67.31 0)
 			(effects
 				(font
@@
 		)
 		(property "Value" "+3.3V"
-			(at 22.86 96.52 0)
+			(at 41.91 58.42 0)
 			(effects
 				(font
@@
 		)
 		(property "Footprint" ""
-			(at 22.86 91.44 0)
+			(at 41.91 63.5 0)
 			(effects
 				(font
@@
 		)
 		(property "Datasheet" ""
-			(at 22.86 91.44 0)
+			(at 41.91 63.5 0)
 			(effects
 				(font
@@
 		)
 		(property "Description" "Power symbol creates a global label with name \"+3.3V\""
-			(at 22.86 91.44 0)
+			(at 41.91 63.5 0)
 			(effects
 				(font
@@
 		)
 		(instances
-			(project ""
+			(project "sensor-board-pressure"
 				(path "/073ec1fb-7e7a-4821-a0d2-1e02de7627d5"
 					(reference "#PWR09")
@@
 	)
 	(symbol
+		(lib_id "Mechanical:MountingHole")
+		(at 139.7 115.57 0)
+		(unit 1)
+		(exclude_from_sim no)
+		(in_bom no)
+		(on_board yes)
+		(dnp no)
+		(fields_autoplaced yes)
+		(property "Reference" "H1"
+			(at 142.24 114.2999 0)
+			(effects
+				(font
+					(size 1.27 1.27)
+				)
+				(justify left)
+			)
+		)
+		(property "Value" "MountingHole"
+			(at 142.24 116.8399 0)
+			(effects
+				(font
+					(size 1.27 1.27)
+				)
+				(justify left)
+			)
+		)
+		(property "Footprint" "MountingHole:MountingHole_2.7mm_M2.5_Pad"
+			(at 139.7 115.57 0)
+			(effects
+				(font
+					(size 1.27 1.27)
+				)
+				(hide yes)
+			)
+		)
+		(property "Datasheet" "~"
+			(at 139.7 115.57 0)
+			(effects
+				(font
+					(size 1.27 1.27)
+				)
+				(hide yes)
+			)
+		)
+		(property "Description" "Mounting Hole without connection"
+			(at 139.7 115.57 0)
+			(effects
+				(font
+					(size 1.27 1.27)
+				)
+				(hide yes)
+			)
+		)
+		(instances
+			(project "sensor-board-pressure"
+				(path "/073ec1fb-7e7a-4821-a0d2-1e02de7627d5"
+					(reference "H1")
+					(unit 1)
+				)
+			)
+		)
+	)
+	(symbol
 		(lib_id "power:+3.3V")
 		(at 86.36 69.85 0)
@@
 	(symbol
 		(lib_id "2026-01-23_05-30-51:C0603C104K5RACTU")
-		(at 22.86 83.82 270)
-		(unit 1)
-		(exclude_from_sim no)
-		(in_bom yes)
-		(on_board yes)
-		(dnp no)
-		(fields_autoplaced yes)
+		(at 41.91 78.74 90)
+		(unit 1)
+		(exclude_from_sim no)
+		(in_bom yes)
+		(on_board yes)
+		(dnp no)
 		(property "Reference" "C1"
-			(at 26.67 86.3599 90)
+			(at 38.354 74.422 90)
 			(effects
 				(font
@@
 		)
 		(property "Value" "100nF"
-			(at 26.67 88.8999 90)
+			(at 39.37 71.628 90)
 			(effects
 				(font
@@
 		)
 		(property "Footprint" "Capacitor_SMD:C_0805_2012Metric"
-			(at 22.86 83.82 0)
+			(at 41.91 78.74 0)
 			(effects
 				(font
@@
 		)
 		(property "Datasheet" "https://content.kemet.com/datasheets/KEM_C1002_X7R_SMD.pdf"
-			(at 22.86 83.82 0)
+			(at 41.91 78.74 0)
 			(effects
 				(font
@@
 		)
 		(property "Description" ""
-			(at 22.86 83.82 0)
-			(effects
-				(font
+			(at 41.91 78.74 0)
+			(effects
+				(font
